File: Circuito/Acionamento BLDC 2023-2/Acionamento BLDC.kicad_sch (KiCad schematic)
At the start: 74 parts, among them J1 55V, J14 Sensores, J2 Motor, J3 Telemetria, J4 Potenciômetro, J5 DM, K1 G5LE-1, Q1 FDH50N50, Q2 FDH50N50, Q3 FDH50N50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

Commit message: Versão 2023-2
Parts:
- removed J10, J11, J12, J13, J6, J7, J8, J9: ~, TestPoint:TestPoint_Loop_D3.50mm_Drill0.9mm_Beaded, symbol Connector:TestPoint_Small
- removed J3: Telemetria, Connector_Phoenix_MC:PhoenixContact_MC_1,5_3-G-3.81_1x03_P3.81mm_Horizontal, symbol Connector:Conn_01x03_Male
- removed K1: G5LE-1, Relay_THT:Relay_SPDT_Omron-G5LE-1, symbol Relay:G5LE-1
- added F1: Fuse 10A, Fuse:Fuse_Blade_ATO_directSolder, symbol Device:Fuse
- added J3: Telemetria, Connector_Phoenix_MC:PhoenixContact_MC_1,5_4-G-3.81_1x04_P3.81mm_Horizontal, symbol Connector:Conn_01x04_Pin
- added J6: Bat, Connector_Phoenix_MSTB:PhoenixContact_MSTBA_2,5_3-G-5,08_1x03_P5.08mm_Horizontal, symbol Connector:Conn_01x03_Pin
- added K2: RAYEX-L90AS, Relay_THT:Relay_SPST_RAYEX-L90AS, symbol Relay:RAYEX-L90AS
- added U9: LM35-LP, Package_TO_SOT_THT:TO-92_Inline, symbol Sensor_Temperature:LM35-LP
- C1: footprint Capacitor_THT:CP_Radial_D8.0mm_P2.50mm -> Capacitor_THT:CP_Radial_D8.0mm_P3.50mm
- C11, C13, C5, C9: footprint Capacitor_THT:CP_Radial_D10.0mm_P3.50mm -> Capacitor_THT:CP_Radial_D8.0mm_P3.50mm
- C15, C16: footprint Capacitor_THT:CP_Radial_D22.0mm_P10.00mm_SnapIn -> Capacitor_THT:CP_Radial_D17.0mm_P7.50mm
- C17: footprint Capacitor_THT:CP_Radial_D8.0mm_P2.50mm -> Capacitor_THT:CP_Radial_D5.0mm_P2.50mm
- C6: value 470u 63V -> 470u 100V; footprint Capacitor_THT:CP_Radial_D13.0mm_P5.00mm -> Capacitor_THT:CP_Radial_D17.0mm_P7.50mm
- D2: value 1N5822 -> SS56; footprint Diode_THT:D_DO-201AD_P15.24mm_Horizontal -> Diode_SMD:D_3220_8050Metric_Pad2.65x5.15mm_HandSolder
- J1: value 55V -> Carga
Connections:
- net +12V: now also J3.1 (Pin_1), U9.1 (+V_{S})
- net BL: now also Q4.1 (G), R10.2
- net CL: now also Q6.1 (G), R12.2
- net FaseB: now also C11.2, U5.6 (VS), U6.3 (-Vo)
- net FaseC: now also C13.2, U7.6 (VS), U8.3 (-Vo)
- net GND: now also J3.4 (Pin_4), J6.3 (Pin_3), K2.A2, U9.3 (GND); no longer J1.1 (Pin_1)
- net TempMot: now also J3.2 (Pin_2)
- net V55+: now also J1.1 (Pin_1), F1.2, K2.14; no longer J1.2 (Pin_2)
- net at C15.1, C16.1, D3.1 (K)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: now also K2.13
- net at J5.2 (Pin_2): now also K2.A1
- new net: J1.2 (Pin_2), J6.1 (Pin_1)
- new net: F1.1, J6.2 (Pin_2)
- new net TempDiss: J3.3 (Pin_3), U9.2 (V_{OUT})
Other:
- note added: "Controle"
- note added: "Potência"
- company: (none) -> Kerschbaumer
- moved on the sheet: C1, C14, C15, C16, C17, C2, C3, C5, C6, C7, C8, D1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
